Commit message: looking

File: hsrb_description/robots/hsrb4s.urdf (robot description, URDF)
Before this commit: robot hsrb, 51 links, 50 joints
Joints:
- joint joint_x: limit lower=-5 upper=5 effort=10000.0 velocity=0.5 -> lower=-10 upper=10 effort=10000.0 velocity=0.5
- joint joint_y: limit lower=-5 upper=5 effort=10000.0 velocity=0.5 -> lower=-10 upper=10 effort=10000.0 velocity=0.5
